File: KiCAD/UNO/UNO.sch (KiCad schematic (older format))
At the start: 8 parts, among them P1 Power, P2 Analog, P3 Digital, P4 Digital, P5 CONN_01X01, P6 CONN_01X01, P7 CONN_01X01, P8 CONN_01X01

Commit message: Adding LED Connectors
Parts:
- removed P5, P6, P7, P8: CONN_01X01, Socket_Arduino_Uno:Arduino_1pin, symbol CONN_01X01
- added J? (x9): Conn_01x03, symbol Conn_01x03
Connections:
- wire segments 38 -> 41
- no-connect marks 5 -> 1
Other:
- note removed: "Holes"
Changed lines of the file:
@@
 LIBS:contrib
 LIBS:valves
-LIBS:Arduino_As_Uno-cache
+LIBS:UNO-cache
 EELAYER 25 0
 EELAYER END
@@
 Text Label 10550 1200 0    60   ~ 0
 A5(SCL)
-Text Notes 10850 1000 0    60   ~ 0
-Holes
 Text Notes 8550 750  0    60   ~ 0
 Shield for Arduino that uses\nthe same pin disposition\nlike "Uno" board Rev 3.
@@
 	1    0    0    -1
 $EndComp
-$Comp
-L CONN_01X01 P5
-U 1 1 56D71177
-P 10800 650
-F 0 "P5" V 10900 650 50  0000 C CNN
-F 1 "CONN_01X01" V 10900 650 50  0001 C CNN
-F 2 "Socket_Arduino_Uno:Arduino_1pin" H 10721 724 20  0000 C CNN
-F 3 "" H 10800 650 50  0000 C CNN
-	1    10800 650
-	0    -1   -1   0
-$EndComp
-$Comp
-L CONN_01X01 P6
-U 1 1 56D71274
-P 10900 650
-F 0 "P6" V 11000 650 50  0000 C CNN
-F 1 "CONN_01X01" V 11000 650 50  0001 C CNN
-F 2 "Socket_Arduino_Uno:Arduino_1pin" H 10900 650 20  0001 C CNN
-F 3 "" H 10900 650 50  0000 C CNN
-	1    10900 650
-	0    -1   -1   0
-$EndComp
-$Comp
-L CONN_01X01 P7
-U 1 1 56D712A8
-P 11000 650
-F 0 "P7" V 11100 650 50  0000 C CNN
-F 1 "CONN_01X01" V 11100 650 50  0001 C CNN
-F 2 "Socket_Arduino_Uno:Arduino_1pin" V 11000 650 20  0001 C CNN
-F 3 "" H 11000 650 50  0000 C CNN
-	1    11000 650
-	0    -1   -1   0
-$EndComp
-$Comp
-L CONN_01X01 P8
-U 1 1 56D712DB
-P 11100 650
-F 0 "P8" V 11200 650 50  0000 C CNN
-F 1 "CONN_01X01" V 11200 650 50  0001 C CNN
-F 2 "Socket_Arduino_Uno:Arduino_1pin" H 11024 572 20  0000 C CNN
-F 3 "" H 11100 650 50  0000 C CNN
-	1    11100 650
-	0    -1   -1   0
-$EndComp
-NoConn ~ 10800 850
-NoConn ~ 10900 850
-NoConn ~ 11000 850
-NoConn ~ 11100 850
 $Comp
 L CONN_01X08 P4
@@
 	10300 1500 10300 3150
 Wire Wire Line
-	9300 2100 9300 2200
-Wire Wire Line
-	9300 2200 9300 3150
+	9300 2100 9300 3150
 Wire Notes Line
 	8500 500  8500 3450
@@
 Text Notes 9700 1600 0    60   ~ 0
 1
-Wire Notes Line
-	11200 1000 10700 1000
-Wire Notes Line
-	10700 1000 10700 500
+$Comp
+L Conn_01x03 J?
+U 1 1 5A859814
+P 1400 1400
+F 0 "J?" H 1400 1600 50  0000 C CNN
+F 1 "Conn_01x03" H 1400 1200 50  0001 C CNN
+F 2 "" H 1400 1400 50  0001 C CNN
+F 3 "" H 1400 1400 50  0001 C CNN
+	1    1400 1400
+	1    0    0    -1
+$EndComp
+$Comp
+L Conn_01x03 J?
+U 1 1 5A859C4D
+P 1400 1950
+F 0 "J?" H 1400 2150 50  0000 C CNN
+F 1 "Conn_01x03" H 1400 1750 50  0001 C CNN
+F 2 "" H 1400 1950 50  0001 C CNN
+F 3 "" H 1400 1950 50  0001 C CNN
+	1    1400 1950
+	1    0    0    -1
+$EndComp
+$Comp
+L Conn_01x03 J?
+U 1 1 5A859C83
+P 1400 2500
+F 0 "J?" H 1400 2700 50  0000 C CNN
+F 1 "Conn_01x03" H 1400 2300 50  0001 C CNN
+F 2 "" H 1400 2500 50  0001 C CNN
+F 3 "" H 1400 2500 50  0001 C CNN
+	1    1400 2500
+	1    0    0    -1
+$EndComp
+$Comp
+L Conn_01x03 J?
+U 1 1 5A859CBE
+P 1400 3050
+F 0 "J?" H 1400 3250 50  0000 C CNN
+F 1 "Conn_01x03" H 1400 2850 50  0001 C CNN
+F 2 "" H 1400 3050 50  0001 C CNN
+F 3 "" H 1400 3050 50  0001 C CNN
+	1    1400 3050
+	1    0    0    -1
+$EndComp
+$Comp
+L Conn_01x03 J?
+U 1 1 5A859CFC
+P 1400 3600
+F 0 "J?" H 1400 3800 50  0000 C CNN
+F 1 "Conn_01x03" H 1400 3400 50  0001 C CNN
+F 2 "" H 1400 3600 50  0001 C CNN
+F 3 "" H 1400 3600 50  0001 C CNN
+	1    1400 3600
+	1    0    0    -1
+$EndComp
+$Comp
+L Conn_01x03 J?
+U 1 1 5A859D39
+P 1400 4150
+F 0 "J?" H 1400 4350 50  0000 C CNN
+F 1 "Conn_01x03" H 1400 3950 50  0001 C CNN
+F 2 "" H 1400 4150 50  0001 C CNN
+F 3 "" H 1400 4150 50  0001 C CNN
+	1    1400 4150
+	1    0    0    -1
+$EndComp
+$Comp
+L Conn_01x03 J?
+U 1 1 5A859D7D
+P 1400 4650
+F 0 "J?" H 1400 4850 50  0000 C CNN
+F 1 "Conn_01x03" H 1400 4450 50  0001 C CNN
+F 2 "" H 1400 4650 50  0001 C CNN
+F 3 "" H 1400 4650 50  0001 C CNN
+	1    1400 4650
+	1    0    0    -1
+$EndComp
+$Comp
+L Conn_01x03 J?
+U 1 1 5A859DD4
+P 1400 5150
+F 0 "J?" H 1400 5350 50  0000 C CNN
+F 1 "Conn_01x03" H 1400 4950 50  0001 C CNN
+F 2 "" H 1400 5150 50  0001 C CNN
+F 3 "" H 1400 5150 50  0001 C CNN
+	1    1400 5150
+	1    0    0    -1
+$EndComp
+$Comp
+L Conn_01x03 J?
+U 1 1 5A859E18
+P 1400 5700
+F 0 "J?" H 1400 5900 50  0000 C CNN
+F 1 "Conn_01x03" H 1400 5500 50  0001 C CNN
+F 2 "" H 1400 5700 50  0001 C CNN
+F 3 "" H 1400 5700 50  0001 C CNN
+	1    1400 5700
+	1    0    0    -1
+$EndComp
+Wire Wire Line
+	1200 1300 1150 1300
+Wire Wire Line
+	1150 1300 1150 1250
+Wire Wire Line
+	1200 1500 1150 1500
+Wire Wire Line
+	1150 1500 1150 1550
+$Comp
+L GND #PWR?
+U 1 1 5A85A676
+P 1150 1550
+F 0 "#PWR?" H 1150 1300 50  0001 C CNN
+F 1 "GND" H 1150 1400 50  0000 C CNN
+F 2 "" H 1150 1550 50  0001 C CNN
+F 3 "" H 1150 1550 50  0001 C CNN
+	1    1150 1550
+	1    0    0    -1
+$EndComp
+$Comp
+L +5V #PWR?
+U 1 1 5A85A6A4
+P 1150 1250
+F 0 "#PWR?" H 1150 1100 50  0001 C CNN
+F 1 "+5V" H 1150 1390 50  0000 C CNN
+F 2 "" H 1150 1250 50  0001 C CNN
+F 3 "" H 1150 1250 50  0001 C CNN
+	1    1150 1250
+	1    0    0    -1
+$EndComp
 $EndSCHEMATC
