File: KiCAD/UNO/UNO.kicad_pcb (KiCad board)
At the start: 2 copper layers, 68.6 x 53.3 mm, 8 parts, among them P1 Power, P2 Analog, P3 Digital, P4 Digital, P5 CONN_01X01, P6 CONN_01X01, P7 CONN_01X01, P8 CONN_01X01

Commit message: 9 LEDs Added and Motor Connector
Parts:
- added J1: Conn_01x03, Socket_Strips:Socket_Strip_Angled_1x03_Pitch2.54mm, F.Cu at (212.6, 66.7)
- added J10: Conn_01x06, Socket_Strips:Socket_Strip_Straight_1x06_Pitch2.54mm, F.Cu at (186.6, 100.3)
- added J2: Conn_01x03, Socket_Strips:Socket_Strip_Angled_1x03_Pitch2.54mm, F.Cu at (202.4, 66.7)
- added J3: Conn_01x03, Socket_Strips:Socket_Strip_Angled_1x03_Pitch2.54mm, F.Cu at (192.3, 66.7)
- added J4: Conn_01x03, Socket_Strips:Socket_Strip_Angled_1x03_Pitch2.54mm, F.Cu at (182.1, 66.7)
- added J5: Conn_01x03, Socket_Strips:Socket_Strip_Angled_1x03_Pitch2.54mm, F.Cu at (172.0, 66.7)
- added J6: Conn_01x03, Socket_Strips:Socket_Strip_Angled_1x03_Pitch2.54mm, F.Cu at (161.8, 66.7)
- added J7: Conn_01x03, Socket_Strips:Socket_Strip_Angled_1x03_Pitch2.54mm, F.Cu at (151.6, 66.7)
- added J8: Conn_01x03, Socket_Strips:Socket_Strip_Angled_1x03_Pitch2.54mm, F.Cu at (141.5, 66.7)
- added J9: Conn_01x03, Socket_Strips:Socket_Strip_Angled_1x03_Pitch2.54mm, F.Cu at (130.7, 66.7)
