File: KiCAD/UNO/UNO.kicad_pcb (KiCad board)
At the start: 2 copper layers, 22 parts, among them J1 Conn_01x04, J10 Conn_01x06, J11 Conn_01x04, J12 Conn_01x02, J13 Conn_01x04, J14 Conn_01x04, J15 Conn_01x04, J16 Conn_01x04, J17 Conn_01x04, J2 Conn_01x04, J3 Conn_01x04, J4 Conn_01x04, J5 Conn_01x04, J6 Conn_01x04, J7 Conn_01x04, J8 Conn_01x04, J9 Conn_01x04, P1 Power, P2 Analog, P3 Digital, P4 Digital, P8 CONN_01X01

Commit message: no message
Parts:
- added J18: Conn_01x02, Pin_Headers:Pin_Header_Straight_1x02_Pitch2.54mm, F.Cu at (-10.2, -4.19)
- added J19: Conn_01x02, Pin_Headers:Pin_Header_Straight_1x02_Pitch2.54mm, F.Cu at (-4.57, 8.51)
- added J20: Conn_01x02, Pin_Headers:Pin_Header_Straight_1x02_Pitch2.54mm, F.Cu at (-17.3, -16.9)
- added J21: Conn_01x02, Pin_Headers:Pin_Header_Straight_1x02_Pitch2.54mm, F.Cu at (31.5, 4.70)
- added J22: Conn_01x02, Pin_Headers:Pin_Header_Straight_1x02_Pitch2.54mm, F.Cu at (22.6, -18.2)
- added J23: Conn_01x02, Pin_Headers:Pin_Header_Straight_1x02_Pitch2.54mm, F.Cu at (4.57, 0.64)
- added J24: Conn_01x02, Pin_Headers:Pin_Header_Straight_1x02_Pitch2.54mm, F.Cu at (13.5, -19.2)
- added J25: Conn_01x02, Pin_Headers:Pin_Header_Straight_1x02_Pitch2.54mm, F.Cu at (10.9, -7.49)
- added J26: Conn_01x02, Pin_Headers:Pin_Header_Straight_1x02_Pitch2.54mm, F.Cu at (121.4, 46.1)
- added R1: R, Resistors_SMD:R_0603_HandSoldering, F.Cu at (35.3, -18.2)
- added R10: R, Resistors_THT:R_Axial_DIN0204_L3.6mm_D1.6mm_P5.08mm_Horizontal, F.Cu at (43.4, -3.94)
- added R11: R, Resistors_SMD:R_0603_HandSoldering, F.Cu at (-27.4, -11.0)
- added R12: R, Resistors_THT:R_Axial_DIN0204_L3.6mm_D1.6mm_P5.08mm_Horizontal, F.Cu at (28.4, -1.40)
- added R13: R, Resistors_SMD:R_0603_HandSoldering, F.Cu at (-19.6, -8.26)
- added R14: R, Resistors_THT:R_Axial_DIN0204_L3.6mm_D1.6mm_P5.08mm_Horizontal, F.Cu at (20.8, 2.67)
- added R15: R, Resistors_SMD:R_0603_HandSoldering, F.Cu at (-19.6, -2.16)
- added R16: R, Resistors_THT:R_Axial_DIN0204_L3.6mm_D1.6mm_P5.08mm_Horizontal, F.Cu at (12.4, 3.17)
- added R17: R, Resistors_SMD:R_0603_HandSoldering, F.Cu at (124.2, 47.4)
- added R18: R, Resistors_THT:R_Axial_DIN0204_L3.6mm_D1.6mm_P5.08mm_Horizontal, F.Cu at (1.27, -20.7)
- added R2: R, Resistors_THT:R_Axial_DIN0204_L3.6mm_D1.6mm_P5.08mm_Horizontal, F.Cu at (32.0, -8.26)
- added R3: R, Resistors_SMD:R_0603_HandSoldering, F.Cu at (-25.9, -2.16)
- added R4: R, Resistors_THT:R_Axial_DIN0204_L3.6mm_D1.6mm_P5.08mm_Horizontal, F.Cu at (118.4, 45.1)
- added R5: R, Resistors_SMD:R_0603_HandSoldering, F.Cu at (-22.6, 4.45)
- added R6: R, Resistors_THT:R_Axial_DIN0204_L3.6mm_D1.6mm_P5.08mm_Horizontal, F.Cu at (-28.2, -17.9)
- added R7: R, Resistors_SMD:R_0603_HandSoldering, F.Cu at (-18.3, 6.73)
- added R8: R, Resistors_THT:R_Axial_DIN0204_L3.6mm_D1.6mm_P5.08mm_Horizontal, F.Cu at (42.7, -13.6)
- added R9: R, Resistors_SMD:R_0603_HandSoldering, F.Cu at (-14.0, 12.1)
Connections:
- net /LED2 renamed Net-(J2-Pad3)
- net /LED3 renamed Net-(J3-Pad3)
- net /LED4 renamed Net-(J4-Pad3)
- net /LED5 renamed Net-(J5-Pad3)
- net /LED6 renamed Net-(J6-Pad3)
- net /LED7 renamed Net-(J7-Pad3)
- net /LED8 renamed Net-(J8-Pad3)
- net /LED9 renamed Net-(J9-Pad3)
- J1 pad 1: Net-(J1-Pad1) -> GND
- J1 pad 4: GND -> Net-(J1-Pad4)
- J2 pad 1: Net-(J2-Pad1) -> GND
- J2 pad 4: GND -> Net-(J19-Pad1)
- J3 pad 1: Net-(J3-Pad1) -> GND
- J3 pad 4: GND -> Net-(J20-Pad1)
- J4 pad 1: Net-(J4-Pad1) -> GND
- J4 pad 4: GND -> Net-(J21-Pad1)
- J5 pad 1: Net-(J5-Pad1) -> GND
- J5 pad 4: GND -> Net-(J22-Pad1)
- J6 pad 1: Net-(J6-Pad1) -> GND
- J6 pad 4: GND -> Net-(J23-Pad1)
- J7 pad 1: Net-(J7-Pad1) -> GND
- J7 pad 4: GND -> Net-(J24-Pad1)
- J8 pad 1: Net-(J8-Pad1) -> GND
- J8 pad 4: GND -> Net-(J25-Pad1)
- J9 pad 1: Net-(J9-Pad1) -> GND
- J9 pad 4: GND -> Net-(J26-Pad1)
